Commit message: fix urdf model orientation and add more tests with quaternion

File: inclinometer/urdf/hwt905_inclinometer.urdf.xacro (robot description, xacro)
@@ -35,5 +35,5 @@
     <parent link="base_footprint"/>
     <child link="base_link"/>
-    <origin xyz="0 0 0" rpy="0 0 0"/>
+    <origin xyz="0 0 0" rpy="0 0 -1.57"/>
   </joint>
   <link name="box_link">
@@ -53,5 +53,5 @@
   </link>
   <joint name="box_joint" type="fixed">
-    <parent link="base_footprint"/>
+    <parent link="base_link"/>
     <child link="box_link"/>
     <origin xyz="0 0 ${INCLINOMETER_BOX_Z/2}" rpy="0 0 0"/>
